Commit message: first

File: xarm_description/urdf/laser_dual_xarm_device.urdf.xacro (robot description, xacro)
@@ -44,8 +44,8 @@
   <xacro:arg name="geometry_type_2" default="box"/>
   <xacro:arg name="geometry_mass_2" default="0.1"/>
-  <xacro:arg name="geometry_height_2" default="0.1"/>
+  <xacro:arg name="geometry_height_2" default="0.01"/>
   <xacro:arg name="geometry_radius_2" default="0.1"/>
-  <xacro:arg name="geometry_length_2" default="0.1"/>
-  <xacro:arg name="geometry_width_2" default="0.1"/>
+  <xacro:arg name="geometry_length_2" default="0.4"/>
+  <xacro:arg name="geometry_width_2" default="0.3"/>
   <xacro:arg name="geometry_mesh_filename_2" default=""/>
   <xacro:arg name="geometry_mesh_origin_xyz_2" default="0 0 0"/>
@@ -59,5 +59,5 @@
   <xacro:arg name="mesh_suffix" default="stl"/>
   <!-- load xarm device -->
-  <xacro:include filename="$(find xarm_description)/urdf/xarm_device_macro.xacro" />
+  <xacro:include filename="$(find xarm_description)/urdf/laser_xarm_device_macro.xacro" />
   <xacro:xarm_device prefix="$(arg prefix_1)" hw_ns="$(arg hw_ns)" limited="$(arg limited)"
     effort_control="$(arg effort_control)" velocity_control="$(arg velocity_control)"
@@ -84,14 +84,14 @@
     ros2_control_plugin="$(arg ros2_control_plugin)" robot_type="$(arg robot_type_2)"
     load_gazebo_plugin="true" ros2_control_params="$(arg ros2_control_params)"
-    attach_to="world" attach_xyz="0 1 0" attach_rpy="0 0 0" create_attach_link="false"
+    attach_to="world" attach_xyz="1.2 0 0" attach_rpy="0 0 3.1416" create_attach_link="false"
     add_realsense_d435i="$(arg add_realsense_d435i_2)"
     add_d435i_links="$(arg add_d435i_links_2)"
-    add_other_geometry="$(arg add_other_geometry_2)"
-    geometry_type="$(arg geometry_type_2)" geometry_mass="$(arg geometry_mass_2)"
-    geometry_height="$(arg geometry_height_2)" geometry_radius="$(arg geometry_radius_2)"
-    geometry_length="$(arg geometry_length_2)" geometry_width="$(arg geometry_width_2)"
+    add_other_geometry="true"
+    geometry_type="box" geometry_mass="0.1"
+    geometry_height="0.01" geometry_radius="$(arg geometry_radius_2)"
+    geometry_length="0.4" geometry_width="0.3"
     geometry_mesh_filename="$(arg geometry_mesh_filename_2)"
     geometry_mesh_origin_xyz="$(arg geometry_mesh_origin_xyz_2)" geometry_mesh_origin_rpy="$(arg geometry_mesh_origin_rpy_2)"
-    geometry_mesh_tcp_xyz="$(arg geometry_mesh_tcp_xyz_2)" geometry_mesh_tcp_rpy="$(arg geometry_mesh_tcp_rpy_2)"
+    geometry_mesh_tcp_xyz="$(arg geometry_mesh_tcp_xyz_2)" geometry_mesh_tcp_rpy="0 1.5708 0"
     robot_ip="$(arg robot_ip_2)" report_type="$(arg report_type_2)"
     baud_checkset="$(arg baud_checkset_2)" default_gripper_baud="$(arg default_gripper_baud_2)"

File: xarm_description/urdf/other/other_geometry.urdf.xacro (robot description, xacro)
@@ -100,5 +100,5 @@
     <link name="${prefix}link_tcp" />
     <joint name="${prefix}joint_tcp" type="fixed">
-      <origin xyz="${_tcp_xyz}" rpy="${_tcp_rpy}" />
+      <origin xyz="${_tcp_xyz}" rpy="${geometry_mesh_tcp_rpy}" />
       <parent link="${prefix}other_geometry_link" />
       <child link="${prefix}link_tcp" />
